Commit message: [launch][configs]
* Revised launch file to correctly load parameters from all config YAMLs and pass it to aerial_robot_core node which sets them on the param server

* Reworked model launch system to pass config and init path with better naming (unsure how RvizInit can be used but it was implement in the old repo)

* Removed inertia of root in urdf since gazebo complained

File: robots/mini_quadrotor/urdf/robot.urdf.xacro (robot description, xacro)
@@ -78,12 +78,4 @@
   <!-- dummy root link for KDL -->
   <link name="root">
-    <inertial>
-      <origin xyz="0 0 0" rpy="0 0 0"/>
-      <mass value="0.00001"/>
-      <inertia
-          ixx="0.000001" ixy="0.0" ixz="0.0"
-          iyy="0.000001" iyz="0.0"
-          izz="0.000002"/>
-    </inertial>
   </link>
   <joint name="root_joint" type="fixed">
