Commit message: [ROS2][Gimbalrotor] Migration of gimbalrotor package from ROS1 to ROS2 (#37)
* [Simulation] Apply rotor thrust commands in Gazebo

* [MiniQuadrotor][simulation] Add rotor effort interfaces

* [Simulation] Run spinal flight modules from attitude controller

* [Control] Make main loop rate warning configurable

* [MiniQuadrotor][simulation] Update simulation bringup parameters

* [MiniQuadrotor][simulation] Tune controller gains

* [Simulation] Feed ground truth attitude to spinal control

* [Simulation] Apply rotor wrenches on parent body links

* [MiniQuadrotor][simulation] Restore rotor visual spin

* [Simulation] Fix clang-format for PR checks

* [CI] Fix ROS distro expansion in lint workflow

* [CI] Fix colcon lint failures

* [Controller][LQI] Fix bug in the gain initialization process of LQI

* [Core][mocap] Add OptiTrack NatNet receiver

* [Estimation][IMU] Allow receive-time stamping for spinal IMU

* [Model] Respect fixed model initialization option

* [Navigation] Improve spinal arming and halt handling

* [MiniQuadrotor][bringup] Launch spinal and mocap on real machine

* [Control][LQI] Throttle repeated activation logs

* [MiniQuadrotor][control] Tune real-machine flight parameters

* [CI] Apply pre-commit fixes

* [CI] Stabilize navigation log formatting

* [Gazebo] Modified gazebo gui setting for WSL2

* Enable configurable flight navigation plugin

* Add ROS 2 gimbalrotor robot package

* Add roll pitch keyboard teleop commands

File: robots/mini_quadrotor/urdf/robot.gazebo.xacro (robot description, xacro)
@@ -3,9 +3,25 @@
     xmlns:xacro="http://www.ros.org/wiki/xacro" name="mini_quadrotor" >
   <xacro:arg name="robot_name" default="mini_quadrotor" />
+  <xacro:arg name="rotor_visual_speed_rate" default="20.0" />
   <!-- robot urdf -->
   <xacro:include filename="$(find mini_quadrotor)/urdf/robot.urdf.xacro" />
+  <xacro:macro name="rotor_control_joint" params="id">
+    <joint name="rotor${id}">
+      <command_interface name="effort">
+        <param name="min">${min_force}</param>
+        <param name="max">${max_force}</param>
+      </command_interface>
+      <state_interface name="position">
+        <param name="initial_value">${0}</param>
+      </state_interface>
+      <state_interface name="velocity"/>
+      <state_interface name="effort"/>
+    </joint>
+  </xacro:macro>
   <ros2_control name="aerial_robot_sim_system" type="system">
     <hardware>
       <plugin>gz_ros2_control/AerialRobotHwSim</plugin>
+      <param name="m_f_rate">${m_f_rate}</param>
+      <param name="rotor_visual_speed_rate">$(arg rotor_visual_speed_rate)</param>
     </hardware>
     <joint name="dummy_joint">
@@ -20,4 +36,8 @@
       <state_interface name="effort"/>
     </joint>
+    <xacro:rotor_control_joint id="1"/>
+    <xacro:rotor_control_joint id="2"/>
+    <xacro:rotor_control_joint id="3"/>
+    <xacro:rotor_control_joint id="4"/>
     <sensor name="spinal_imu">
       <state_interface name="orientation.x"/>

File: robots/mini_quadrotor/urdf/robot.urdf.xacro (robot description, xacro)
@@ -5,4 +5,5 @@
   <baselink name="fc" />
   <thrust_link name="thrust" />
+  <xacro:arg name="rotor_joint_velocity_limit" default="10000.0" />
   <!-- kinematics [m] -->
   <xacro:property name="rotor_x" value="0.085" />
@@ -10,7 +11,9 @@
   <xacro:property name="rotor_z" value="0.026" />
   <!-- dynamics -->
-  <m_f_rate value="-0.011" /> <!-- drag torque rate -->
+  <xacro:property name="m_f_rate" value="-0.011" /> <!-- drag torque rate -->
+  <m_f_rate value="${m_f_rate}" />
   <xacro:property name="max_force" value="8.0" /> <!-- [N] -->
   <xacro:property name="min_force" value="0.0" /> <!-- [N] -->
+  <xacro:property name="rotor_joint_velocity_limit" value="$(arg rotor_joint_velocity_limit)" />
   <!-- friction -->
   <xacro:macro name="damping_factor" params="link">
@@ -39,5 +42,5 @@
   <xacro:macro name="propeller_module" params="id x y z direction">
     <joint name="rotor${id}" type="continuous">
-      <limit effort="100.0" lower="${min_force}" upper="${max_force}" velocity="0.5"/>
+      <limit effort="100.0" lower="${min_force}" upper="${max_force}" velocity="${rotor_joint_velocity_limit}"/>
       <parent link="main_body"/>
       <child link="thrust${id}"/>
